Commit message: 1-26-2021 update

File: main env/1.15hole.urdf (robot description, URDF)
Before this commit: robot 1.15in squarehole.SLDPRT, 1 links, 0 joints
Links:
- removed link 1.15in squarehole.SLDPRT
- added link 1.15in squarehole_C.SLDPRT, mass 0.36078; collision mesh filename=package://1.15in squarehole_C.SLDPRT/meshes/1.15in squareho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; visual mesh filename=package://1.15in squarehole_C.SLDPRT/meshes/1.15in squareho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

File: main env/1.15in squarehole_C.SLDPRT/urdf/1.15in squarehole_C.SLDPRT.urdf (robot description, URDF)
Before this commit: robot 1.25in squarehole.SLDPRT, 1 links, 0 joints
Links:
- removed link 1.25in squarehole.SLDPRT
- added link 1.15in squarehole_C.SLDPRT, mass 0.36078; collision mesh filename=package://1.15in squarehole_C.SLDPRT/meshes/1.15in squareho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; visual mesh filename=package://1.15in squarehole_C.SLDPRT/meshes/1.15in squareho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

File: main env/1.25hole.urdf (robot description, URDF)
Before this commit: robot 1.25in squarehole.SLDPRT, 1 links, 0 joints
Links:
- removed link 1.25in squarehole.SLDPRT
- added link 1.25in squarehole_C.SLDPRT, mass 0.35488; collision mesh filename=package://1.25in squarehole_C.SLDPRT/meshes/1.25in squareho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; visual mesh filename=package://1.25in squarehole_C.SLDPRT/meshes/1.25in squareho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

File: main env/1.25in squarehole_C.SLDPRT/urdf/1.25in squarehole_C.SLDPRT.urdf (robot description, URDF)
Before this commit: robot 1in rectangular block.SLDPRT, 1 links, 0 joints
Links:
- removed link 1in rectangular block.SLDPRT
- added link 1.25in squarehole_C.SLDPRT, mass 0.35488; collision mesh filename=package://1.25in squarehole_C.SLDPRT/meshes/1.25in squareho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; visual mesh filename=package://1.25in squarehole_C.SLDPRT/meshes/1.25in squareho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

File: main env/1.5hole.urdf (robot description, URDF)
Before this commit: robot 1.5in squarehole, 1 links, 0 joints
Links:
- removed link 1.5in squarehole
- added link 1.5in squarehole_C.SLDPRT, mass 0.33798; collision mesh filename=package://1.5in squarehole_C.SLDPRT/meshes/1.5in squarehole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; visual mesh filename=package://1.5in squarehole_C.SLDPRT/meshes/1.5in squarehole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

File: main env/1.5in squarehole_C.SLDPRT/urdf/1.5in squarehole_C.SLDPRT.urdf (robot description, URDF)
Before this commit: robot 1.15in squarehole.SLDPRT, 1 links, 0 joints
Links:
- removed link 1.15in squarehole.SLDPRT
- added link 1.5in squarehole_C.SLDPRT, mass 0.33798; collision mesh filename=package://1.5in squarehole_C.SLDPRT/meshes/1.5in squarehole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; visual mesh filename=package://1.5in squarehole_C.SLDPRT/meshes/1.5in squarehole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

File: main env/1block.urdf (robot description, URDF)
Before this commit: robot 1in rectangular block.SLDPRT, 1 links, 0 joints
Links:
- removed link 1in rectangular block.SLDPRT
- added link 1in rectangular block_C.SLDPRT, mass 0.049161; collision mesh filename=package://1in rectangular block_C.SLDPRT/meshes/1in rectang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; visual mesh filename=package://1in rectangular block_C.SLDPRT/meshes/1in rectang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

File: main env/1in rectangular block_C.SLDPRT/urdf/1in rectangular block_C.SLDPRT.urdf (robot description, URDF)
Before this commit: robot 1.5in squarehole, 1 links, 0 joints
Links:
- removed link 1.5in squarehole
- added link 1in rectangular block_C.SLDPRT, mass 0.049161; collision mesh filename=package://1in rectangular block_C.SLDPRT/meshes/1in rectang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; visual mesh filename=package://1in rectangular block_C.SLDPRT/meshes/1in rectang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

Commit message: 2-4-2021 update

File: main env/1.15hole.urdf (robot description, URDF)
Before this commit: robot 1.15in squarehole_C.SLDPRT, 1 links, 0 joints
Links:
- removed link 1.15in squarehole_C.SLDPRT
- added link 1.15hole, mass 0.36078; collision mesh filename=package://1.15hole/meshes/1.15hole.STL; visual mesh filename=package://1.15hole/meshes/1.15hole.STL

File: main env/1.25hole.urdf (robot description, URDF)
Before this commit: robot 1.25in squarehole_C.SLDPRT, 1 links, 0 joints
Links:
- removed link 1.25in squarehole_C.SLDPRT
- added link 1.25hole, mass 0.35488; collision mesh filename=package://1.25hole/meshes/1.25hole.STL; visual mesh filename=package://1.25hole/meshes/1.25hole.STL

File: main env/1.5hole.urdf (robot description, URDF)
Before this commit: robot 1.5in squarehole_C.SLDPRT, 1 links, 0 joints
Links:
- removed link 1.5in squarehole_C.SLDPRT
- added link 1.5hole, mass 0.33798; collision mesh filename=package://1.5hole/meshes/1.5hole.STL; visual mesh filename=package://1.5hole/meshes/1.5hole.STL

File: main env/combined.urdf (robot description, URDF)
Before this commit: robot , 2 links, 1 joints
Links:
- removed link 1.5in squarehole_C.SLDPRT
- added link 1.5hole, mass 0.33798; collision mesh filename=./1.5hole/meshes/1.5hole.STL scale=1.00000 1.00000 1.00000; visual mesh filename=./1.5hole/meshes/1.5hole.STL scale=1.00000 1.00000 1.00000
Joints:
- joint joint_dummy1: child 1.5in squarehole_C.SLDPRT -> 1.5hole
